File: lego_robot.sch (KiCad schematic (older format))
At the start: 29 parts, among them J1 Motor_Connector, J2 Motor_Connector, J3 Motor_Connector, U1 ShengYang-BMS, U2 DSN-1504-3A, U3 L80-M39, U4 STM32-NUCLEO-F446RE, U5 ICM-20948, U6 BD65496MUV, U7 BD65496MUV, U8 BD65496MUV

Commit message: More work on schematic
Parts:
- removed TP? (x4): TestPoint, symbol Connector:TestPoint
- added C6: 100nF, symbol Device:C
- added D2: LED, symbol Device:LED
- added J1: Battery_Connector, symbol lego_robot:Battery_Connector
- added J2: Barrel_Jack_MountingPin, symbol Connector:Barrel_Jack_MountingPin
- added JP1, JP2: Jumper_NC_Dual, symbol Device:Jumper_NC_Dual
- added NT1: NT_GND, symbol Device:Net-Tie_3
- added NT2: NT_MOTOR_PWR, symbol Device:Net-Tie_2
- added R1, R2: R, symbol Device:R
- added TP1: TP_VBAT_S3, symbol Connector:TestPoint
- added TP10: TP_GPS_UART_RX, symbol Connector:TestPoint
- added TP11: TP_GPS_UART_TX, symbol Connector:TestPoint
- added TP12: TP_GPS_RESET, symbol Connector:TestPoint
- added TP2: TP_VBAT_S2, symbol Connector:TestPoint
- added TP3: TP_VBAT_S1, symbol Connector:TestPoint
- added TP4: TP_CHGR_P, symbol Connector:TestPoint
- added TP5: TP_CHGR_N, symbol Connector:TestPoint
- added TP7: TP_LOGIC_3V3, symbol Connector:TestPoint
- added TP8: TP_LOGIC_5V, symbol Connector:TestPoint
- added TP9: TP_LOGIC_GND, symbol Connector:TestPoint
- C1: value C -> 10uF
- C10: renamed from C7; value C -> 10uF
- C11: renamed from C8; value C -> 10uF
- C12: renamed from C9; value C -> 10uF
- C2: value C -> 100nF
- C3: renamed from C10; value C -> 100nF
- C4: renamed from C3; value C -> 10uF
- C5: renamed from C11; value C -> 100nF
- C7: renamed from C4; value C -> 100nF
- C8: renamed from C5; value C -> 100nF
- C9: renamed from C6; value C -> 100nF
- TP13: renamed from TP2; value TestPoint -> TP_VBAT_REG
- TP6: renamed from TP1; value TestPoint -> TP_VBAT
- gave numbers to parts that had none: 1
- renumbered J1 to J3, J2 to J4, J3 to J5, U4 to U1, U1 to U2, U2 to U3, U5 to U4, U3 to U5
Connections:
- net labels added: CHGR_N, CHGR_P, LOGIC_3V3, LOGIC_5V, MOTOR_MODE, MOTOR_TR1, MOTOR_TR2, VBAT_REG, VBAT_S1, VBAT_S2, VBAT_S3, ~MOTOR1_PS, ~MOTOR2_PS, ~MOTOR3_PS
- net labels removed: LOGIC_VIN, VBAT_UNREG
- wire segments 115 -> 167
- no-connect marks 2 -> 19
Other:
- note added: "<- to periphs"
- note added: "from PSU -> \n\n"
- moved on the sheet: C1, C10, C2, C3, C4, C5, C7, C8, C9, D1, J3, J4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
